File: hardware/controller/controller.kicad_pcb (KiCad board)
At the start: 2 copper layers, 16 parts, among them J1 ADC_CONN, J2 CONN_07, J3 USB_MICRO-B_FEMALE-SMT, J4 JST_2MM_MALE, U1 MCP73831, U2 BL652

Commit message: feat: finish controller pcb
Parts:
- removed SWD_VCC1: VCC, PAD.03X.05
- added C3: 1.0UF-0402-16V-10%, 0402, F.Cu at (236.0, 128.5)
- added R5: 1MOHM-0603-1_4W-5%, 0603, F.Cu at (235.4, 139.4)
- added R6: 1MOHM-0603-1_4W-5%, 0603, F.Cu at (238.8, 139.4)
- added U3: TC1014, Silicon-Standard:SOT23-5, F.Cu at (233.0, 133.3)
- added USB: HRO-TYPE-C-31-M-12, deps:HRO-TYPE-C-31-M-12-HandSoldering_modified, F.Cu at (209.3, 131.8)
- D1: footprint LED-0603 -> LED:LED-0603
- J1: footprint 1X03 -> Connectors:1X03
- J2: value CONN_07 -> DISP_CONN; footprint 1X07 -> Connectors:1X07
- J3: value USB_MICRO-B_FEMALE-SMT -> BATT_CONN; footprint USB-B-MICRO-SMD -> 1X02
- J4: value JST_2MM_MALE -> SHUTDOWN; footprint JST-2-SMD -> 1X02
- R1: value RESISTOR0402 -> 5.1K
- R2: value 2K -> RESISTOR0402
- R3: value RESISTOR0402 -> 2K
- SWD_CLK1: value SWDCLK -> CLK; footprint PAD.03X.05 -> Connectors:PAD.03X.05
- SWD_GND1: footprint PAD.03X.05 -> Connectors:PAD.03X.05
- SWD_IO1: value SWDIO -> IO; footprint PAD.03X.05 -> Connectors:PAD.03X.05
- U1: footprint SOT23-5 -> Silicon-Standard:SOT23-5
- moved SWD_IO1 112.2 mm to (248.3, 139.1), turned to 180 degrees
- moved SWD_CLK1 107.5 mm to (245.7, 139.1), turned to 180 degrees
- moved SWD_GND1 102.8 mm to (243.2, 139.1), turned to 180 degrees
- moved U2 101.8 mm to (244.3, 131.8), turned to 180 degrees
- moved C2 94.1 mm to (223.5, 135.9), turned to 180 degrees
- moved J1 70.5 mm to (222.2, 124.5)
- moved J2 69.5 mm to (230.5, 124.5)
- moved R3 54.4 mm to (222.9, 133.3)
- moved J4 53.7 mm to (231.8, 139.1), turned to 180 degrees
- moved D1 53.1 mm to (226.9, 127.7)
- moved U1 48.1 mm to (226.7, 132.7), turned to 90 degrees
- moved R1 47.8 mm to (220.2, 132.0)
- moved R2 43.7 mm to (223.5, 128.3), turned to 270 degrees
- moved J3 40.5 mm to (222.2, 139.1), turned to 0 degrees
- moved C1 35.3 mm to (221.0, 128.0), turned to 90 degrees
Connections:
- C1 pad 1: Net-(C1-Pad1) -> V_USB
- C2 pad 1: VCC -> V_BATT
- J4 pad 1: GND -> Net-(J4-Pad1)
- J4 pad 2: VCC -> GND
- R1 pad 1: Net-(D1-PadA) -> /CC
- R1 pad 2: Net-(C1-Pad1) -> GND
- R2 pad 1: Net-(R2-Pad1) -> Net-(D1-PadA)
- R2 pad 2: GND -> V_USB
- R3 pad 1: Net-(R2-Pad1) -> Net-(R3-Pad1)
- U1 pad 3: VCC -> V_BATT
- U1 pad 4: Net-(C1-Pad1) -> V_USB
- U1 pad 5: Net-(R2-Pad1) -> Net-(R3-Pad1)
- U2 pad 2: /CS -> Net-(U2-Pad2)
- U2 pad 28: Net-(U2-Pad28) -> /MOSI
- U2 pad 29: Net-(U2-Pad29) -> /SCK
- U2 pad 3: /MOSI -> Net-(U2-Pad3)
- U2 pad 30: Net-(U2-Pad30) -> /DC
- U2 pad 31: Net-(U2-Pad31) -> /RST
- U2 pad 32: Net-(U2-Pad32) -> /CS
- U2 pad 36: /RST -> Net-(U2-Pad36)
- U2 pad 37: /DC -> Net-(U2-Pad37)
- U2 pad 38: /SCK -> Net-(U2-Pad38)
Routing:
- net V_BATT: track 0.00 -> 22.6 mm
- net VCC: track 0.00 -> 22.5 mm
- net V_USB: track 0.00 -> 18.2 mm
- net /AIN0: track 0.00 -> 13.9 mm, vias 0 -> 2
- net /AIN1: track 0.00 -> 10.7 mm
- net Net-(D1-PadC): track 0.00 -> 8.25 mm, vias 0 -> 2
- net /CC: track 0.00 -> 6.50 mm
- net /CS: track 0.00 -> 5.29 mm
- net Net-(J4-Pad1): track 0.00 -> 4.82 mm
- net /MOSI: track 0.00 -> 4.35 mm
- net /RST: track 0.00 -> 3.50 mm
- net /SCK: track 0.00 -> 3.04 mm
- net /SWDIO: track 0.00 -> 2.87 mm
- net /SWDCLK: track 0.00 -> 2.70 mm
- net Net-(D1-PadA): track 0.00 -> 2.55 mm
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- added copper zone on B.Cu, net GND
- added copper zone on F.Cu, net GND
Other:
- board outline added: 41.9 x 18.4 mm
