File: hardware/receiver/receiver.sch (KiCad schematic (older format))
At the start: 7 parts, among them J1 CONN_04, U1 BL652

Commit message: feat: finish controller pcb
Parts:
- C1: symbol SparkFun-Capacitors:0.1UF-0402-16V-10% -> receiver-rescue:0.1UF-0402-16V-10%-SparkFun-Capacitors
- GND1, SWDCLK1, SWDIO1, VCC1: symbol SparkFun-Connectors:TEST-POINT3 -> receiver-rescue:TEST-POINT3-SparkFun-Connectors
- J1: symbol SparkFun-Connectors:CONN_04 -> receiver-rescue:CONN_04-SparkFun-Connectors
- U1: symbol RF_Bluetooth:BL652 -> receiver-rescue:BL652-RF_Bluetooth
Changed lines of the file:
@@
 $EndDescr
 $Comp
-L RF_Bluetooth:BL652 U1
+L receiver-rescue:BL652-RF_Bluetooth U1
 U 1 1 5C65B55E
 P 5600 3750
@@
 $EndComp
 $Comp
-L SparkFun-PowerSymbols:GND #GND0101
+L receiver-rescue:GND-SparkFun-PowerSymbols #GND0101
 U 1 1 5C65B751
 P 5800 5100
@@
 $EndComp
 $Comp
-L SparkFun-PowerSymbols:VCC #SUPPLY0101
+L receiver-rescue:VCC-SparkFun-PowerSymbols #SUPPLY0101
 U 1 1 5C65B87F
 P 5950 2450
@@
 $EndComp
 $Comp
-L SparkFun-Connectors:TEST-POINT3 SWDCLK1
+L receiver-rescue:TEST-POINT3-SparkFun-Connectors SWDCLK1
 U 1 1 5C65CA5C
 P 6750 2850
@@
 $EndComp
 $Comp
-L SparkFun-Connectors:TEST-POINT3 SWDIO1
+L receiver-rescue:TEST-POINT3-SparkFun-Connectors SWDIO1
 U 1 1 5C65CAD9
 P 6750 2950
@@
 	5950 2650 5950 2450
 $Comp
-L SparkFun-Connectors:CONN_04 J1
+L receiver-rescue:CONN_04-SparkFun-Connectors J1
 U 1 1 5C65D49D
 P 3500 3650
@@
 $EndComp
 $Comp
-L SparkFun-PowerSymbols:VCC #SUPPLY0102
+L receiver-rescue:VCC-SparkFun-PowerSymbols #SUPPLY0102
 U 1 1 5C65D53A
 P 3700 3250
@@
 	3700 3350 3700 3250
 $Comp
-L SparkFun-PowerSymbols:GND #GND0102
+L receiver-rescue:GND-SparkFun-PowerSymbols #GND0102
 U 1 1 5C65DC87
 P 3950 3550
@@
 	4450 3650 4600 3650
 $Comp
-L SparkFun-Connectors:TEST-POINT3 GND1
+L receiver-rescue:TEST-POINT3-SparkFun-Connectors GND1
 U 1 1 5C65F07A
 P 5600 5100
@@
 $EndComp
 $Comp
-L SparkFun-Connectors:TEST-POINT3 VCC1
+L receiver-rescue:TEST-POINT3-SparkFun-Connectors VCC1
 U 1 1 5C65F511
 P 6050 2650
@@
 	3950 3450 3950 3550
 $Comp
-L SparkFun-Capacitors:0.1UF-0402-16V-10% C1
+L receiver-rescue:0.1UF-0402-16V-10%-SparkFun-Capacitors C1
 U 1 1 5C6B209A
 P 8050 3800
@@
 $EndComp
 $Comp
-L SparkFun-PowerSymbols:GND #GND01
+L receiver-rescue:GND-SparkFun-PowerSymbols #GND01
 U 1 1 5C6B248D
 P 8050 4000
@@
 $EndComp
 $Comp
-L SparkFun-PowerSymbols:VCC #SUPPLY01
+L receiver-rescue:VCC-SparkFun-PowerSymbols #SUPPLY01
 U 1 1 5C6B2911
 P 8050 3500
